File: Shiftregister.sch (KiCad schematic (older format))
At the start: 54 parts, among them P1 CONN_01X06, P10 CONN_01X08, P11 CONN_01X08, P12 CONN_01X08, P13 CONN_01X08, P14 CONN_01X08, P15 CONN_01X08, P16 CONN_01X08, P17 CONN_01X08, P18 CONN_01X06, P19 CONN_01X08, P2 CONN_01X08, P3 CONN_01X08, P4 CONN_01X08, P5 CONN_01X08, P6 CONN_02X08, P7 CONN_01X08, P8 CONN_01X08, P9 CONN_01X08, U1 74HC595, U10 74HC595, U11 74HC595, U12 74HC595, U13 74HC595, U14 74HC595, U15 74HC595, U16 74HC595, U2 74HC595, U3 74HC595, U4 74HC595, U5 74HC595, U6 74HC595, U7 74HC595, U8 74HC595, U9 74HC595

Commit message: Added BOM
Parts:
- C1, C10, C11, C12, C13, C14, C15, C16, C17, C3, C4, C5, C6, C7, C8, C9: value CP1 -> 10UF
- C2: value CP1 -> 100UF
Changed lines of the file:
@@
 P 3250 900
 F 0 "C3" H 3275 1000 50  0000 L CNN
-F 1 "CP1" H 3275 800 50  0000 L CNN
+F 1 "10UF" H 3275 800 50  0000 L CNN
 F 2 "Capacitors_Tantalum_SMD:CP_Tantalum_Case-X_EIA-7343-43_Reflow" H 3250 900 50  0001 C CNN
 F 3 "" H 3250 900 50  0000 C CNN
@@
 P 6850 950
 F 0 "C1" H 6875 1050 50  0000 L CNN
-F 1 "CP1" H 6875 850 50  0000 L CNN
+F 1 "10UF" H 6875 850 50  0000 L CNN
 F 2 "Capacitors_Tantalum_SMD:CP_Tantalum_Case-X_EIA-7343-43_Reflow" H 6850 950 50  0001 C CNN
 F 3 "" H 6850 950 50  0000 C CNN
@@
 P 10250 950
 F 0 "C4" H 10275 1050 50  0000 L CNN
-F 1 "CP1" H 10275 850 50  0000 L CNN
+F 1 "10UF" H 10275 850 50  0000 L CNN
 F 2 "Capacitors_Tantalum_SMD:CP_Tantalum_Case-X_EIA-7343-43_Reflow" H 10250 950 50  0001 C CNN
 F 3 "" H 10250 950 50  0000 C CNN
@@
 P 13650 1050
 F 0 "C5" H 13675 1150 50  0000 L CNN
-F 1 "CP1" H 13675 950 50  0000 L CNN
+F 1 "10UF" H 13675 950 50  0000 L CNN
 F 2 "Capacitors_Tantalum_SMD:CP_Tantalum_Case-X_EIA-7343-43_Reflow" H 13650 1050 50  0001 C CNN
 F 3 "" H 13650 1050 50  0000 C CNN
@@
 P 13650 3350
 F 0 "C9" H 13675 3450 50  0000 L CNN
-F 1 "CP1" H 13675 3250 50  0000 L CNN
+F 1 "10UF" H 13675 3250 50  0000 L CNN
 F 2 "Capacitors_Tantalum_SMD:CP_Tantalum_Case-X_EIA-7343-43_Reflow" H 13650 3350 50  0001 C CNN
 F 3 "" H 13650 3350 50  0000 C CNN
@@
 P 10300 3350
 F 0 "C8" H 10325 3450 50  0000 L CNN
-F 1 "CP1" H 10325 3250 50  0000 L CNN
+F 1 "10UF" H 10325 3250 50  0000 L CNN
 F 2 "Capacitors_Tantalum_SMD:CP_Tantalum_Case-X_EIA-7343-43_Reflow" H 10300 3350 50  0001 C CNN
 F 3 "" H 10300 3350 50  0000 C CNN
@@
 P 3100 3250
 F 0 "C6" H 3125 3350 50  0000 L CNN
-F 1 "CP1" H 3125 3150 50  0000 L CNN
+F 1 "10UF" H 3125 3150 50  0000 L CNN
 F 2 "Capacitors_Tantalum_SMD:CP_Tantalum_Case-X_EIA-7343-43_Reflow" H 3100 3250 50  0001 C CNN
 F 3 "" H 3100 3250 50  0000 C CNN
@@
 P 6800 3300
 F 0 "C7" H 6825 3400 50  0000 L CNN
-F 1 "CP1" H 6825 3200 50  0000 L CNN
+F 1 "10UF" H 6825 3200 50  0000 L CNN
 F 2 "Capacitors_Tantalum_SMD:CP_Tantalum_Case-X_EIA-7343-43_Reflow" H 6800 3300 50  0001 C CNN
 F 3 "" H 6800 3300 50  0000 C CNN
@@
 P 6650 5550
 F 0 "C11" H 6675 5650 50  0000 L CNN
-F 1 "CP1" H 6675 5450 50  0000 L CNN
+F 1 "10UF" H 6675 5450 50  0000 L CNN
 F 2 "Capacitors_Tantalum_SMD:CP_Tantalum_Case-X_EIA-7343-43_Reflow" H 6650 5550 50  0001 C CNN
 F 3 "" H 6650 5550 50  0000 C CNN
@@
 P 10150 5600
 F 0 "C13" H 10175 5700 50  0000 L CNN
-F 1 "CP1" H 10175 5500 50  0000 L CNN
+F 1 "10UF" H 10175 5500 50  0000 L CNN
 F 2 "Capacitors_Tantalum_SMD:CP_Tantalum_Case-X_EIA-7343-43_Reflow" H 10150 5600 50  0001 C CNN
 F 3 "" H 10150 5600 50  0000 C CNN
@@
 P 13550 5550
 F 0 "C12" H 13575 5650 50  0000 L CNN
-F 1 "CP1" H 13575 5450 50  0000 L CNN
+F 1 "10UF" H 13575 5450 50  0000 L CNN
 F 2 "Capacitors_Tantalum_SMD:CP_Tantalum_Case-X_EIA-7343-43_Reflow" H 13550 5550 50  0001 C CNN
 F 3 "" H 13550 5550 50  0000 C CNN
@@
 P 10200 7850
 F 0 "C16" H 10225 7950 50  0000 L CNN
-F 1 "CP1" H 10225 7750 50  0000 L CNN
+F 1 "10UF" H 10225 7750 50  0000 L CNN
 F 2 "Capacitors_Tantalum_SMD:CP_Tantalum_Case-X_EIA-7343-43_Reflow" H 10200 7850 50  0001 C CNN
 F 3 "" H 10200 7850 50  0000 C CNN
@@
 P 13600 7950
 F 0 "C17" H 13625 8050 50  0000 L CNN
-F 1 "CP1" H 13625 7850 50  0000 L CNN
+F 1 "10UF" H 13625 7850 50  0000 L CNN
 F 2 "Capacitors_Tantalum_SMD:CP_Tantalum_Case-X_EIA-7343-43_Reflow" H 13600 7950 50  0001 C CNN
 F 3 "" H 13600 7950 50  0000 C CNN
@@
 P 6700 7850
 F 0 "C15" H 6725 7950 50  0000 L CNN
-F 1 "CP1" H 6725 7750 50  0000 L CNN
+F 1 "10UF" H 6725 7750 50  0000 L CNN
 F 2 "Capacitors_Tantalum_SMD:CP_Tantalum_Case-X_EIA-7343-43_Reflow" H 6700 7850 50  0001 C CNN
 F 3 "" H 6700 7850 50  0000 C CNN
@@
 P 3100 5500
 F 0 "C10" H 3125 5600 50  0000 L CNN
-F 1 "CP1" H 3125 5400 50  0000 L CNN
+F 1 "10UF" H 3125 5400 50  0000 L CNN
 F 2 "Capacitors_Tantalum_SMD:CP_Tantalum_Case-X_EIA-7343-43_Reflow" H 3100 5500 50  0001 C CNN
 F 3 "" H 3100 5500 50  0000 C CNN
@@
 P 2950 7800
 F 0 "C14" H 2975 7900 50  0000 L CNN
-F 1 "CP1" H 2975 7700 50  0000 L CNN
+F 1 "10UF" H 2975 7700 50  0000 L CNN
 F 2 "Capacitors_Tantalum_SMD:CP_Tantalum_Case-X_EIA-7343-43_Reflow" H 2950 7800 50  0001 C CNN
 F 3 "" H 2950 7800 50  0000 C CNN
@@
 P 1750 950
 F 0 "C2" H 1775 1050 50  0000 L CNN
-F 1 "CP1" H 1775 850 50  0000 L CNN
+F 1 "100UF" H 1775 850 50  0000 L CNN
 F 2 "Capacitors_Tantalum_SMD:CP_Tantalum_Case-X_EIA-7343-43_Reflow" H 1750 950 50  0001 C CNN
 F 3 "" H 1750 950 50  0000 C CNN

Commit message: fiddle
Parts:
- R1: value R -> 220k
Changed lines of the file:
@@
 P 1225 2075
 F 0 "R1" V 1305 2075 50  0000 C CNN
-F 1 "R" V 1225 2075 50  0000 C CNN
+F 1 "220k" V 1225 2075 50  0000 C CNN
 F 2 "Resistors_SMD:R_0805_HandSoldering" V 1155 2075 50  0001 C CNN
 F 3 "" H 1225 2075 50  0000 C CNN
